File: Hardware/BMU/BMU.kicad_pcb (KiCad board)
At the start: 2 copper layers, 80 x 17.8 mm, 29 parts, among them IC1 HY2213-BB3A, J1 USB_C_Receptacle_PowerOnly_6P, J2 Conn_01x05_Pin, Q1 FS8205A, Q2 AO3401A, Q3 BUK7880-55A, U1 DW01A, U2 TP4056

Commit message: Updated BMU
Parts:
- added TP1: TestPoint, TestPoint:TestPoint_Plated_Hole_D2.0mm, F.Cu at (101.6, 59.7)
Routing:
- net PMOS-Drain: track 75.7 -> 69.9 mm
- net Net-(U2-PROG): track 10.8 -> 13.1 mm
- net Net-(U2-GND): track 45.6 -> 43.4 mm
- net GND: track 7.14 -> 5.12 mm
- net Net-(IC1-OUT): track 66.4 -> 68.2 mm
- net Net-(IC1-VSS): track 105.6 -> 104.7 mm
- net Net-(U1-OC): track 35.5 -> 36.4 mm
- net Net-(D2-K): track 7.19 -> 8.06 mm
- net Net-(D1-K): track 20.2 -> 20.9 mm
- net Net-(U1-VCC): track 18.2 -> 17.5 mm
- net +5V: track 98.9 -> 99.5 mm
- net Net-(J2-Pin_4): track 18.1 -> 18.7 mm
- added copper zone on B.Cu, net GND
Other:
- outline, holes or cut-outs redrawn
