File: Hardware/Controller-BMU-Kombi/_autosave-Controller-BMU-Kombi.kicad_sch (KiCad schematic)
At the start: 18 parts, among them J1 Conn_01x05_Socket, J2 Conn_01x05_Socket, J3 Conn_01x05_Socket, J4 Conn_01x05_Socket, J5 Conn_01x05_Socket, J6 Conn_01x05_Socket

Commit message: Updates
Parts:
- U2: footprint (none) -> Batteriestecker:Batteriestecker
Changed lines of the file:
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@@
 			)
 		)
-		(property "Footprint" ""
+		(property "Footprint" "Batteriestecker:Batteriestecker"
 			(at 185.42 121.92 0)
 			(effects
