File: Hardware/Controller-BMU-Kombi/_autosave-Controller-BMU-Kombi.kicad_pcb (KiCad board)
At the start: 2 copper layers, 15 parts, among them J1 Conn_01x05_Socket, J2 Conn_01x05_Socket, J3 Conn_01x05_Socket, J4 Conn_01x05_Socket, J5 Conn_01x05_Socket, J6 Conn_01x05_Socket, U2 ESP32_NODEMCU

Commit message: updates
Parts:
- moved U8 9.22 mm to (62.3, 104.1)
Changed lines of the file:
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@@
 	(footprint "Batteriestecker:Batteriestecker"
 		(layer "F.Cu")
-		(at 53.38 101.64)
+		(at 62.27 104.1)
 		(property "Reference" "U8"
 			(at 0 -0.5 0)
